File: wr-rusefi.sch (KiCad schematic (older format))
At the start: 30 parts, among them P101 USB_OTG, P102 CONN_02X20, U101 ISL89410, U102 ISL89410, U103 FT230XS, U104 STM32F373CCTx, U105 MCP2562-E/SN, U106 LD1117S33TR, U107 MAX9924

Commit message: Rework most of board for rusefi
Parts:
- removed P102: CONN_02X20, Pin_Headers:Pin_Header_Straight_2x20, symbol CONN_02X20
- removed U104: STM32F373CCTx, Housings_QFP:LQFP-48_7x7mm_Pitch0.5mm, symbol STM32F373CCTx
- added C101: 1nF, Capacitors_SMD:C_0603_HandSoldering, symbol C
- added C102, C103: 20pF, Capacitors_SMD:C_0603_HandSoldering, symbol C
- added C112, C113: 2.2uF, Capacitors_SMD:C_0603_HandSoldering, symbol C
- added C114, C115, C116: .1uF, Capacitors_SMD:C_0603_HandSoldering, symbol C
- added C117: 4.7uF, Capacitors_SMD:C_0603_HandSoldering, symbol C
- added P102, P103, P105, P106: CONN_01X08, Socket_Strips:Socket_Strip_Straight_1x08, symbol CONN_01X08
- added P104: CONN_01X04, Socket_Strips:Socket_Strip_Straight_1x04, symbol CONN_01X04
- added P107: CONN_01X02, Socket_Strips:Socket_Strip_Straight_1x02, symbol CONN_01X02
- added R110, R111, R112: 10k, Resistors_SMD:R_0603_HandSoldering, symbol R
- added U104: MAX9924, wr-efi:uMAX-10, symbol MAX9924
- added U108, U110: ISL89410, Housings_SOIC:SOIC-8_3.9x4.9mm_Pitch1.27mm, symbol ISL89410
- added U109: STM32F407VGTx, Housings_QFP:LQFP-100_14x14mm_Pitch0.5mm, symbol STM32F407VGTx
- added Y101: Crystal, Crystals:Crystal_HC52-6mm_Vertical, symbol Crystal
Connections:
- net +3V3: now also C114.1, C115.1, C116.1, C117.1, R112.2, U109.100 (VDD), U109.11 (VDD), U109.19 (VDD), U109.21 (VREF+), U109.22 (VDDA), U109.28 (VDD), U109.50 (VDD), U109.6 (VBAT), U109.75 (VDD)
- net +5V: now also U104.10 (VCC), U108.6 (V+), U110.6 (V+)
- net AIN0: now also P102.1 (P1); no longer C111.30 (B20)
- net AIN1: now also P102.2 (P2); no longer C111.20 (B10)
- net AIN2: now also P102.3 (P3); no longer C111.29 (B19)
- net AIN3: now also P102.4 (P4); no longer C111.19 (B9)
- net AIN4: now also P102.5 (P5); no longer C111.28 (B18)
- net AIN5: now also P102.6 (P6); no longer C111.18 (B8)
- net AIN6: now also P102.7 (P7); no longer C111.27 (B17)
- net AIN7: now also P102.8 (P8); no longer C111.17 (B7)
- net CANH: now also P107.1 (P1); no longer C111.14 (B4)
- net CANL: now also P107.2 (P2); no longer C111.24 (B14)
- net CAN_RX: now also U109.51 (CAN2_RX/ETH_TXD0/I2C2_SMBA/I2S2_WS/SPI2_NSS/TIM1_BKIN/USART3_CK/USB_OTG_HS_ID/USB_OTG_HS_ULPI_D5/PB12)
- net CAN_TX: now also U109.92 (CAN2_TX/DCMI_D5/I2C1_SCL/TIM4_CH1/USART1_TX/PB6)
- net GND: now also C102.2, C103.2, C112.2, C113.2, C114.2, C115.2, C116.2, C117.2, U104.4 (BIAS), U104.5 (GND), U104.6 (ZERO_EN), U104.9 (INT_THRS), U108.3 (GND), U109.10 (VSS), U109.20 (VSSA), U109.27 (VSS), U109.74 (VSS), U109.99 (VSS), U110.3 (GND)
- net IGN_A_IN: now also U109.48 (ADC1_EXTI11/ADC2_EXTI11/ADC3_EXTI11/ETH_TX_EN/I2C2_SDA/TIM2_CH4/USART3_RX/USB_OTG_HS_ULPI_D4/PB11)
- net IGN_A_OUT: now also P105.1 (P1); no longer C111.11 (B1)
- net IGN_B_IN: now also U109.47 (ETH_RX_ER/I2C2_SCL/I2S2_CK/SPI2_SCK/TIM2_CH3/USART3_TX/USB_OTG_HS_ULPI_D3/PB10)
- net IGN_B_OUT: now also P105.2 (P2); no longer C111.12 (B2)
- net IGN_C_IN: now also U109.46 (PE15/ADC1_EXTI15/ADC2_EXTI15/ADC3_EXTI15/FSMC_D12/FSMC_DA12/TIM1_BKIN)
- net IGN_C_OUT: now also P105.3 (P3); no longer C111.21 (B11)
- net IGN_D_IN: now also U109.45 (PE14/FSMC_D11/FSMC_DA11/TIM1_CH4)
- net IGN_D_OUT: now also P105.4 (P4); no longer C111.22 (B12)
- net INJ_A_IN: now also U109.54 (ADC1_EXTI15/ADC2_EXTI15/ADC3_EXTI15/I2S2_SD/RTC_REFIN/SPI2_MOSI/TIM12_CH2/TIM1_CH3N/TIM8_CH3N/USB_OTG_HS_DP/PB15)
- net INJ_B_IN: now also U109.53 (I2S2_ext_SD/SPI2_MISO/TIM12_CH1/TIM1_CH2N/TIM8_CH2N/USART3_RTS/USB_OTG_HS_DM/PB14)
- net a0: now also U109.15 (ADC1_IN10/ADC2_IN10/ADC3_IN10/USB_OTG_HS_ULPI_STP/PC0)
- net a1: now also U109.16 (ADC1_IN11/ADC2_IN11/ADC3_IN11/ETH_MDC/PC1)
- net a2: now also U109.17 (ADC1_IN12/ADC2_IN12/ADC3_IN12/ETH_TXD2/I2S2_ext_SD/SPI2_MISO/USB_OTG_HS_ULPI_DIR/PC2)
- net a3: now also U109.18 (ADC1_IN13/ADC2_IN13/ADC3_IN13/ETH_TX_CLK/I2S2_SD/SPI2_MOSI/USB_OTG_HS_ULPI_NXT/PC3)
- net a4: now also U109.23 (ADC1_IN0/ADC2_IN0/ADC3_IN0/ETH_CRS/SYS_WKUP/TIM2_CH1/TIM2_ETR/TIM5_CH1/TIM8_ETR/UART4_TX/USART2_CTS/PA0)
- net a5: now also U109.24 (ADC1_IN1/ADC2_IN1/ADC3_IN1/ETH_REF_CLK/ETH_RX_CLK/TIM2_CH2/TIM5_CH2/UART4_RX/USART2_RTS/PA1)
- net a6: now also U109.25 (ADC1_IN2/ADC2_IN2/ADC3_IN2/ETH_MDIO/TIM2_CH3/TIM5_CH3/TIM9_CH1/USART2_TX/PA2)
- net a7: now also U109.26 (ADC1_IN3/ADC2_IN3/ADC3_IN3/ETH_COL/TIM2_CH4/TIM5_CH4/TIM9_CH2/USART2_RX/USB_OTG_HS_ULPI_D0/PA3)
- net ftdi_rx: now also U109.78 (DCMI_D8/I2S3_CK/SDIO_D2/SPI3_SCK/UART4_TX/USART3_TX/PC10)
- net ftdi_tx: now also U109.79 (ADC1_EXTI11/ADC2_EXTI11/ADC3_EXTI11/DCMI_D4/I2S3_ext_SD/SDIO_D3/SPI3_MISO/UART4_RX/USART3_RX/PC11)
- net ls_1: now also U109.55 (PD8/FSMC_D13/FSMC_DA13/USART3_TX)
- net ls_2: now also U109.56 (PD9/DAC_EXTI9/FSMC_D14/FSMC_DA14/USART3_RX)
- net ls_3: now also U109.57 (PD10/FSMC_D15/FSMC_DA15/USART3_CK)
- net ls_4: now also U109.58 (PD11/ADC1_EXTI11/ADC2_EXTI11/ADC3_EXTI11/FSMC_A16/FSMC_CLE/USART3_CTS)
- net at CONN_SWD101.2 (P2): now also U109.72 (SYS_JTMS-SWDIO/PA13)
- net at CONN_SWD101.3 (P3): now also U109.76 (SYS_JTCK-SWCLK/PA14)
- net at C109.1, R108.1, R109.2: now also U109.29 (ADC1_IN4/ADC2_IN4/DAC_OUT1/DCMI_HSYNC/I2S3_WS/SPI1_NSS/SPI3_NSS/USART2_CK/USB_OTG_HS_SOF/PA4)
- net VR+: no longer names the net of C111.23 (B13)
- net VR+: now also P103.3 (P3); no longer R105.2
- net VR-: no longer names the net of C111.13 (B3)
- net VR-: now also P103.4 (P4); no longer R106.2
- net VRIN renamed VRIN1
- net VRIN1: now also U109.63 (DCMI_D0/I2S2_MCK/SDIO_D6/TIM3_CH1/TIM8_CH1/USART6_TX/PC6)
- new net: C111.11 (B1), P103.8 (P8)
- new net: C111.12 (B2), P103.6 (P6)
- new net: C111.14 (B4), P103.2 (P2)
- new net: C111.17 (B7), P106.8 (P8)
- new net: C111.18 (B8), P106.6 (P6)
- new net: C111.19 (B9), P106.4 (P4)
- new net: C111.20 (B10), P106.2 (P2)
- new net: C111.21 (B11), P103.7 (P7)
- new net: C111.22 (B12), P103.5 (P5)
- new net: C111.24 (B14), P103.1 (P1)
- new net: C111.27 (B17), P106.7 (P7)
- new net: C111.28 (B18), P106.5 (P5)
- new net: C111.29 (B19), P106.3 (P3)
- new net: C111.30 (B20), P106.1 (P1)
- new net: C102.1, U109.12 (PH0/RCC_OSC_IN), Y101.2
- new net: C103.1, U109.13 (PH1/RCC_OSC_OUT), Y101.1
- new net: C112.1, U109.49 (VCAP_1)
- new net: C113.1, U109.73 (VCAP_2)
- new net: C101.1, R110.1, U104.1 (IN+)
- new net: C101.2, R111.1, U104.2 (IN-)
- new net IGN_E_IN: U108.2 (INA), U109.44 (PE13/FSMC_D10/FSMC_DA10/TIM1_CH3)
- new net IGN_E_OUT: P105.5 (P5), U108.7 (OUTA)
- new net IGN_F_IN: U108.4 (INB), U109.43 (PE12/FSMC_D9/FSMC_DA9/TIM1_CH3N)
- new net IGN_F_OUT: P105.6 (P6), U108.5 (OUTB)
- new net IGN_G_IN: U109.42 (PE11/ADC1_EXTI11/ADC2_EXTI11/ADC3_EXTI11/FSMC_D8/FSMC_DA8/TIM1_CH2), U110.2 (INA)
- new net IGN_G_OUT: P105.7 (P7), U110.7 (OUTA)
- new net IGN_H_IN: U109.41 (PE10/FSMC_D7/FSMC_DA7/TIM1_CH2N), U110.4 (INB)
- new net IGN_H_OUT: P105.8 (P8), U110.5 (OUTB)
- new net VR1+: P104.1 (P1), R105.2
- new net VR1-: P104.2 (P2), R106.2
- new net VR2+: P104.3 (P3), R110.2
- new net VR2-: P104.4 (P4), R111.2
- new net VRIN2: R112.1, U104.7 (COUT), U109.30 (ADC1_IN5/ADC2_IN5/DAC_OUT2/SPI1_SCK/TIM2_CH1/TIM2_ETR/TIM8_CH1N/USB_OTG_HS_ULPI_CK/PA5)
- no-connect marks 41 -> 11

Commit message: Board mostly complete
Parts:
- removed CONN_SWD101: CONN_01X03, Pin_Headers:Pin_Header_Straight_1x03, symbol CONN_01X03
- added P108: USB_OTG, Connect:USB_Mini-B, symbol USB_OTG
- added P109: CONN_01X02, Socket_Strips:Socket_Strip_Straight_1x02, symbol CONN_01X02
- added P110: CONN_01X06, Socket_Strips:Socket_Strip_Straight_1x06, symbol CONN_01X06
- added R113: 10k, Resistors_SMD:R_0603_HandSoldering, symbol R
- Y101: footprint Crystals:Crystal_HC52-6mm_Vertical -> Crystals:Crystal_HC49-U_Vertical
Connections:
- net +3V3: now also P109.2 (P2), P110.1 (P1), R113.1
- net GND: now also P108.5 (GND), P108.6 (shield), P110.3 (P3)
- net ls_1: now also U109.58 (PD11/ADC1_EXTI11/ADC2_EXTI11/ADC3_EXTI11/FSMC_A16/FSMC_CLE/USART3_CTS); no longer U109.55 (PD8/FSMC_D13/FSMC_DA13/USART3_TX)
- net ls_4: now also U109.55 (PD8/FSMC_D13/FSMC_DA13/USART3_TX); no longer U109.58 (PD11/ADC1_EXTI11/ADC2_EXTI11/ADC3_EXTI11/FSMC_A16/FSMC_CLE/USART3_CTS)
- net NRST: now reaches R101.2
- net NRST: now also U109.14 (NRST), P110.5 (P5)
- net at U109.72 (SYS_JTMS-SWDIO/PA13): now also P110.4 (P4)
- net at U109.76 (SYS_JTCK-SWCLK/PA14): now also P110.2 (P2)
- net at U109.68 (DAC_EXTI9/DCMI_D0/I2C3_SMBA/TIM1_CH2/USART1_TX/USB_OTG_FS_VBUS/PA9): now also P108.1 (VCC)
- net at U109.70 (ADC1_EXTI11/ADC2_EXTI11/ADC3_EXTI11/CAN1_RX/TIM1_CH4/USART1_CTS/USB_OTG_FS_DM/PA11): now also P108.2 (D-)
- net at U109.71 (CAN1_TX/TIM1_ETR/USART1_RTS/USB_OTG_FS_DP/PA12): now also P108.3 (D+)
- net at U109.94 (BOOT0): now also P109.1 (P1), R113.2
- no-connect marks 11 -> 59

Commit message: Add debug LEDs, power via 2nd USB
Parts:
- added D103: PMEG2010EA, Diodes_SMD:D_SOD-323_HandSoldering, symbol D_Schottky
- added D104, D105, D106, D107, D108: LED, LEDs:LED_0603, symbol LED
- added R114, R115, R116, R117, R118: 1k, Resistors_SMD:R_0603_HandSoldering, symbol R
Connections:
- net +3V3: now also R114.2
- net +5V: now also D103.1 (K)
- net GND: now also D104.1 (K), D105.1 (K), D106.1 (K), D107.1 (K), D108.1 (K)
- net PD12: now reaches U109.59 (PD12/FSMC_A17/FSMC_ALE/TIM4_CH1/USART3_RTS)
- net PD12: now also R115.2
- net PD13: now reaches U109.60 (PD13/FSMC_A18/TIM4_CH2)
- net PD13: now also R116.2
- net PD14: now reaches U109.61 (PD14/FSMC_D0/FSMC_DA0/TIM4_CH3)
- net PD14: now also R117.2
- net PD15: now reaches U109.62 (PD15/ADC1_EXTI15/ADC2_EXTI15/ADC3_EXTI15/FSMC_D1/FSMC_DA1/TIM4_CH4)
- net PD15: now also R118.2
- net at P108.1 (VCC), U109.68 (DAC_EXTI9/DCMI_D0/I2C3_SMBA/TIM1_CH2/USART1_TX/USB_OTG_FS_VBUS/PA9): now also D103.2 (A)
- new net: D104.2 (A), R114.1
- new net: D108.2 (A), R118.1
- new net: D107.2 (A), R117.1
- new net: D106.2 (A), R116.1
- new net: D105.2 (A), R115.1
- no-connect marks 59 -> 55

Commit message: cleanup
Connections:
- net BATT_ADC: now reaches C109.1, R108.1, R109.2, U109.29 (ADC1_IN4/ADC2_IN4/DAC_OUT1/DCMI_HSYNC/I2S3_WS/SPI1_NSS/SPI3_NSS/USART2_CK/USB_OTG_HS_SOF/PA4)
- net VBUS: now reaches D103.2 (A), P108.1 (VCC), U109.68 (DAC_EXTI9/DCMI_D0/I2C3_SMBA/TIM1_CH2/USART1_TX/USB_OTG_FS_VBUS/PA9)
- net USB_DM: now reaches P108.2 (D-), U109.70 (ADC1_EXTI11/ADC2_EXTI11/ADC3_EXTI11/CAN1_RX/TIM1_CH4/USART1_CTS/USB_OTG_FS_DM/PA11)
- net USB_DP: now reaches P108.3 (D+), U109.71 (CAN1_TX/TIM1_ETR/USART1_RTS/USB_OTG_FS_DP/PA12)
- net SWDIO: now reaches P110.4 (P4), U109.72 (SYS_JTMS-SWDIO/PA13)
- net SWCLK: now reaches P110.2 (P2), U109.76 (SYS_JTCK-SWCLK/PA14)
Changed lines of the file:
@@
 	1    0    0    -1
 $EndComp
-Text GLabel 12900 5600 2    60   Input ~ 0
+Text GLabel 12700 5600 2    60   Input ~ 0
 a0
-Text GLabel 12900 5700 2    60   Input ~ 0
+Text GLabel 12700 5700 2    60   Input ~ 0
 a1
-Text GLabel 12900 5800 2    60   Input ~ 0
+Text GLabel 12700 5800 2    60   Input ~ 0
 a2
-Text GLabel 12900 5900 2    60   Input ~ 0
+Text GLabel 12700 5900 2    60   Input ~ 0
 a3
-Text GLabel 12900 2200 2    60   Input ~ 0
+Text GLabel 12650 2200 2    60   Input ~ 0
 a4
-Text GLabel 12900 2300 2    60   Input ~ 0
+Text GLabel 12650 2300 2    60   Input ~ 0
 a5
-Text GLabel 12900 2400 2    60   Input ~ 0
+Text GLabel 12650 2400 2    60   Input ~ 0
 a6
-Text GLabel 12900 2500 2    60   Input ~ 0
+Text GLabel 12650 2500 2    60   Input ~ 0
 a7
 Text GLabel 1100 10050 0    60   Input ~ 0
@@
 Text GLabel 20600 4150 2    60   Input ~ 0
 ftdi_rx
-Text GLabel 12650 6600 2    60   Input ~ 0
+Text GLabel 12700 6600 2    60   Input ~ 0
 ftdi_rx
-Text GLabel 12650 6700 2    60   Input ~ 0
+Text GLabel 12700 6700 2    60   Input ~ 0
 ftdi_tx
 $Comp
@@
 Text GLabel 1700 5900 2    60   Input ~ 0
 a7
-Text GLabel 12900 4500 2    60   Input ~ 0
+Text GLabel 12700 4500 2    60   Input ~ 0
 CAN_TX
-Text GLabel 12900 5100 2    60   Input ~ 0
+Text GLabel 12700 5100 2    60   Input ~ 0
 CAN_RX
 $Comp
@@
 	1    0    0    -1
 $EndComp
-Text GLabel 12900 4900 2    60   Input ~ 0
+Text GLabel 12700 4900 2    60   Input ~ 0
 IGN_B_IN
 Text GLabel 3200 5400 0    60   Input ~ 0
@@
 L GND #PWR146
 U 1 1 585370D4
-P 13850 3100
-F 0 "#PWR146" H 13850 2850 50  0001 C CNN
-F 1 "GND" H 13850 2950 50  0000 C CNN
-F 2 "" H 13850 3100 50  0000 C CNN
-F 3 "" H 13850 3100 50  0000 C CNN
-	1    13850 3100
+P 19350 2200
+F 0 "#PWR146" H 19350 1950 50  0001 C CNN
+F 1 "GND" H 19350 2050 50  0000 C CNN
+F 2 "" H 19350 2200 50  0000 C CNN
+F 3 "" H 19350 2200 50  0000 C CNN
+	1    19350 2200
 	1    0    0    -1
 $EndComp
@@
 L +12V #PWR145
 U 1 1 5853781A
-P 13850 2100
-F 0 "#PWR145" H 13850 1950 50  0001 C CNN
-F 1 "+12V" H 13850 2240 50  0000 C CNN
-F 2 "" H 13850 2100 50  0000 C CNN
-F 3 "" H 13850 2100 50  0000 C CNN
-	1    13850 2100
+P 19350 1200
+F 0 "#PWR145" H 19350 1050 50  0001 C CNN
+F 1 "+12V" H 19350 1340 50  0000 C CNN
+F 2 "" H 19350 1200 50  0000 C CNN
+F 3 "" H 19350 1200 50  0000 C CNN
+	1    19350 1200
 	1    0    0    -1
 $EndComp
@@
 L R R109
 U 1 1 58539C71
-P 13850 2850
-F 0 "R109" V 13930 2850 50  0000 C CNN
-F 1 "10k" V 13850 2850 50  0000 C CNN
-F 2 "Resistors_SMD:R_0603_HandSoldering" V 13780 2850 50  0001 C CNN
-F 3 "" H 13850 2850 50  0000 C CNN
-	1    13850 2850
+P 19350 1950
+F 0 "R109" V 19430 1950 50  0000 C CNN
+F 1 "10k" V 19350 1950 50  0000 C CNN
+F 2 "Resistors_SMD:R_0603_HandSoldering" V 19280 1950 50  0001 C CNN
+F 3 "" H 19350 1950 50  0000 C CNN
+	1    19350 1950
 	-1   0    0    1
 $EndComp
@@
 L R R108
 U 1 1 5853AA87
-P 13850 2350
-F 0 "R108" V 13930 2350 50  0000 C CNN
-F 1 "100k" V 13850 2350 50  0000 C CNN
-F 2 "Resistors_SMD:R_0603_HandSoldering" V 13780 2350 50  0001 C CNN
-F 3 "" H 13850 2350 50  0000 C CNN
-	1    13850 2350
+P 19350 1450
+F 0 "R108" V 19430 1450 50  0000 C CNN
+F 1 "100k" V 19350 1450 50  0000 C CNN
+F 2 "Resistors_SMD:R_0603_HandSoldering" V 19280 1450 50  0001 C CNN
+F 3 "" H 19350 1450 50  0000 C CNN
+	1    19350 1450
 	-1   0    0    1
 $EndComp
@@
 L C C109
 U 1 1 5853D645
-P 13450 2850
-F 0 "C109" H 13475 2950 50  0000 L CNN
-F 1 "0.01uF" H 13475 2750 50  0000 L CNN
-F 2 "Capacitors_SMD:C_0603_HandSoldering" H 13488 2700 50  0001 C CNN
-F 3 "" H 13450 2850 50  0000 C CNN
-	1    13450 2850
+P 18950 1950
+F 0 "C109" H 18975 2050 50  0000 L CNN
+F 1 "0.01uF" H 18975 1850 50  0000 L CNN
+F 2 "Capacitors_SMD:C_0603_HandSoldering" H 18988 1800 50  0001 C CNN
+F 3 "" H 18950 1950 50  0000 C CNN
+	1    18950 1950
 	1    0    0    -1
 $EndComp
@@
 	1    0    0    -1
 $EndComp
-Text GLabel 12900 6200 2    60   Input ~ 0
+Text GLabel 12700 6200 2    60   Input ~ 0
 VRIN1
 Text GLabel 12650 2700 2    60   Input ~ 0
@@
 	1    0    0    -1
 $EndComp
-Text GLabel 12900 5000 2    60   Input ~ 0
+Text GLabel 12700 5000 2    60   Input ~ 0
 IGN_A_IN
 Text GLabel 3200 5200 0    60   Input ~ 0
@@
 Text GLabel 3200 4900 0    60   Input ~ 0
 IGN_H_IN
-Text GLabel 12900 5400 2    60   Input ~ 0
+Text GLabel 12700 5400 2    60   Input ~ 0
 INJ_A_IN
-Text GLabel 12900 5300 2    60   Input ~ 0
+Text GLabel 12700 5300 2    60   Input ~ 0
 INJ_B_IN
 Text GLabel 3250 6700 0    60   Input ~ 0
@@
 $EndComp
 Wire Wire Line
-	2800 1800 2800 1700
+	2800 1700 2800 1800
 Wire Wire Line
 	19750 3650 19750 3750
@@
 	1250 5800 1450 5800
 Wire Wire Line
-	12450 5100 12900 5100
-Wire Wire Line
-	12900 4500 12450 4500
+	12450 5100 12700 5100
+Wire Wire Line
+	12700 4500 12450 4500
 Wire Wire Line
 	8250 8700 8400 8700
@@
 	2550 10350 2800 10350
 Wire Wire Line
-	12450 5600 12900 5600
-Wire Wire Line
-	12900 5700 12450 5700
-Wire Wire Line
-	12450 5800 12900 5800
-Wire Wire Line
-	12900 5900 12450 5900
-Wire Wire Line
-	12450 2200 12900 2200
-Wire Wire Line
-	12900 2300 12450 2300
-Wire Wire Line
-	12450 2400 12900 2400
-Wire Wire Line
-	12900 2500 12450 2500
+	12450 5600 12700 5600
+Wire Wire Line
+	12700 5700 12450 5700
+Wire Wire Line
+	12450 5800 12700 5800
+Wire Wire Line
+	12700 5900 12450 5900
+Wire Wire Line
+	12450 2200 12650 2200
+Wire Wire Line
+	12650 2300 12450 2300
+Wire Wire Line
+	12450 2400 12650 2400
+Wire Wire Line
+	12650 2500 12450 2500
 Wire Wire Line
 	19850 8900 19850 8800
@@
 Connection ~ 9650 8800
 Wire Wire Line
-	13850 2500 13850 2700
-Connection ~ 13850 2600
-Wire Wire Line
-	13850 3000 13850 3100
-Wire Wire Line
-	13850 2200 13850 2100
-Wire Wire Line
-	13450 2700 13450 2600
-Connection ~ 13450 2600
-Wire Wire Line
-	13450 3000 13450 3050
-Wire Wire Line
-	13450 3050 13850 3050
-Connection ~ 13850 3050
+	19350 1600 19350 1800
+Connection ~ 19350 1700
+Wire Wire Line
+	19350 2100 19350 2200
+Wire Wire Line
+	19350 1300 19350 1200
+Wire Wire Line
+	18950 1800 18950 1700
+Connection ~ 18950 1700
+Wire Wire Line
+	18950 2100 18950 2150
+Wire Wire Line
+	18950 2150 19350 2150
+Connection ~ 19350 2150
 Wire Wire Line
 	7650 1700 7650 1600
@@
 	21650 4750 20350 4750
 Wire Wire Line
-	12650 6600 12450 6600
-Wire Wire Line
-	12450 6700 12650 6700
+	12700 6600 12450 6600
+Wire Wire Line
+	12450 6700 12700 6700
 Connection ~ 7950 1600
 Wire Wire Line
@@
 Connection ~ 8050 1600
 Wire Wire Line
-	12900 6200 12450 6200
-Wire Wire Line
-	12450 2600 13850 2600
+	12700 6200 12450 6200
+Wire Wire Line
+	18700 1700 19350 1700
 Wire Wire Line
 	12650 2700 12450 2700
@@
 	17350 10250 17500 10250
 Wire Wire Line
-	12900 4900 12450 4900
-Wire Wire Line
-	12450 5000 12900 5000
+	12700 4900 12450 4900
+Wire Wire Line
+	12450 5000 12700 5000
 Wire Wire Line
 	3200 5400 3450 5400
@@
 	3200 5200 3450 5200
 Wire Wire Line
-	12450 5300 12900 5300
-Wire Wire Line
-	12900 5400 12450 5400
+	12450 5300 12700 5300
+Wire Wire Line
+	12700 5400 12450 5400
 Wire Wire Line
 	3450 6500 3250 6500
@@
 	0    1    1    0
 $EndComp
-Wire Wire Line
-	12450 3400 14750 3400
-Wire Wire Line
-	14750 3300 12450 3300
-Wire Wire Line
-	12450 3100 12750 3100
-Wire Wire Line
-	12750 3100 12750 3250
-Wire Wire Line
-	12750 3250 14600 3250
-Wire Wire Line
-	14600 3250 14600 3050
-Wire Wire Line
-	14600 3200 14750 3200
 $Comp
 L GND #PWR148
@@
 $EndComp
 Wire Wire Line
-	3450 2400 2350 2400
+	2350 2400 3450 2400
 Wire Wire Line
 	2350 2300 2700 2300
@@
 Wire Wire Line
 	14800 5050 15050 5050
-Wire Wire Line
-	15050 4950 14200 4950
-Wire Wire Line
-	14200 4950 14200 3600
-Wire Wire Line
-	14200 3600 12450 3600
-Wire Wire Line
-	12450 3500 14100 3500
-Wire Wire Line
-	14100 3500 14100 5150
-Wire Wire Line
-	14100 5150 15050 5150
 Wire Wire Line
 	15050 5250 14600 5250
@@
 	0    1    1    0
 $EndComp
-Connection ~ 14600 3200
 $Comp
 L +5V #PWR147
@@
 Wire Wire Line
 	3450 6800 3250 6800
+Text GLabel 18700 1700 0    60   Input ~ 0
+BATT_ADC
+Text GLabel 12650 2600 2    60   Input ~ 0
+BATT_ADC
+Wire Wire Line
+	12650 2600 12450 2600
+Text GLabel 12650 3500 2    60   Input ~ 0
+SWDIO
+Wire Wire Line
+	12650 3500 12450 3500
+Text GLabel 14600 5150 0    60   Input ~ 0
+SWDIO
+Wire Wire Line
+	14600 5150 15050 5150
+Text GLabel 12650 3600 2    60   Input ~ 0
+SWCLK
+Wire Wire Line
+	12650 3600 12450 3600
+Text GLabel 14600 4950 0    60   Input ~ 0
+SWCLK
+Wire Wire Line
+	14600 4950 15050 4950
+Text GLabel 12650 3100 2    60   Input ~ 0
+VBUS
+Wire Wire Line
+	12650 3100 12450 3100
+Text GLabel 12650 3300 2    60   Input ~ 0
+USB_DM
+Text GLabel 12650 3400 2    60   Input ~ 0
+USB_DP
+Wire Wire Line
+	12450 3300 12650 3300
+Wire Wire Line
+	12450 3400 12650 3400
+Text GLabel 14500 3300 0    60   Input ~ 0
+USB_DM
+Text GLabel 14500 3400 0    60   Input ~ 0
+USB_DP
+Wire Wire Line
+	14750 3300 14500 3300
+Wire Wire Line
+	14500 3400 14750 3400
+Text GLabel 14350 3200 0    60   Input ~ 0
+VBUS
+Wire Wire Line
+	14350 3200 14750 3200
+Wire Wire Line
+	14600 3050 14600 3200
+Connection ~ 14600 3200
 $EndSCHEMATC

Commit message: Add reverse protection diode, board cleanup
Parts:
- added D109: D_Schottky, Diodes_SMD:D_SMC_Standard, symbol D_Schottky
Connections:
- net +12V: now also D109.1 (K); no longer C111.6 (A6)
- new net: C111.6 (A6), D109.2 (A)

Commit message: minor layout
Parts:
- added R119, R120, R121, R122: 5k, Resistors_SMD:R_0805_HandSoldering, symbol R
- R105, R106, R110, R111: value 10k -> 5k; footprint Resistors_SMD:R_0603_HandSoldering -> Resistors_SMD:R_0805_HandSoldering
Connections:
- net VR2-: now also R119.2; no longer R111.2
- net at C106.1, U107.1 (IN+): now also R120.1; no longer R105.1
- net at C106.2, U107.2 (IN-): now also R121.1; no longer R106.1
- net at C101.1, U104.1 (IN+): now also R122.1; no longer R110.1
- new net: R111.2, R119.1
- new net: R110.1, R122.2
- new net: R106.1, R121.2
- new net: R105.1, R120.2

Commit message: start redoing layout, lowside drivers and analog routed
Parts:
- RR101: footprint Resistors_ThroughHole:Resistor_Array_SIP9 -> Resistors_ThroughHole:R_Array_SIP9

Commit message: Mostly done new layout
Connections:
- net ls_1: now also U109.56 (PD9/DAC_EXTI9/FSMC_D14/FSMC_DA14/USART3_RX); no longer U109.58 (PD11/ADC1_EXTI11/ADC2_EXTI11/ADC3_EXTI11/FSMC_A16/FSMC_CLE/USART3_CTS)
- net ls_2: now also U109.55 (PD8/FSMC_D13/FSMC_DA13/USART3_TX); no longer U109.56 (PD9/DAC_EXTI9/FSMC_D14/FSMC_DA14/USART3_RX)
- net ls_3: now also U109.58 (PD11/ADC1_EXTI11/ADC2_EXTI11/ADC3_EXTI11/FSMC_A16/FSMC_CLE/USART3_CTS); no longer U109.57 (PD10/FSMC_D15/FSMC_DA15/USART3_CK)
- net ls_4: now also U109.57 (PD10/FSMC_D15/FSMC_DA15/USART3_CK); no longer U109.55 (PD8/FSMC_D13/FSMC_DA13/USART3_TX)
Changed lines of the file:
@@
 Text GLabel 12700 5300 2    60   Input ~ 0
 INJ_B_IN
+Text GLabel 3250 6500 0    60   Input ~ 0
+ls_1
+Text GLabel 3250 6400 0    60   Input ~ 0
+ls_2
 Text GLabel 3250 6700 0    60   Input ~ 0
-ls_1
-Text GLabel 3250 6500 0    60   Input ~ 0
-ls_2
+ls_3
 Text GLabel 3250 6600 0    60   Input ~ 0
-ls_3
-Text GLabel 3250 6400 0    60   Input ~ 0
 ls_4
 $Comp
