File: wr-rusefi.sch (KiCad schematic (older format))
At the start: 70 parts, among them P101 USB_OTG, P102 CONN_01X08, P103 CONN_01X08, P104 CONN_01X04, P105 CONN_01X08, P106 CONN_01X08, P107 CONN_01X02, P108 USB_OTG, P109 CONN_01X02, P110 CONN_01X06, U101 ISL89410, U102 ISL89410, U103 FT230XS, U104 MAX9924, U105 MCP2562-E/SN, U106 LD1117S33TR, U107 MAX9924, U108 ISL89410, U109 STM32F407VGTx, U110 ISL89410, Y101 Crystal

Commit message: Move CAN to PD0/1, nearly done routing
Connections:
- net +3V3: no longer R113.1
- net CAN_RX: now also U109.81 (PD0/CAN1_RX/FSMC_D2/FSMC_DA2); no longer U109.51 (CAN2_RX/ETH_TXD0/I2C2_SMBA/I2S2_WS/SPI2_NSS/TIM1_BKIN/USART3_CK/USB_OTG_HS_ID/USB_OTG_HS_ULPI_D5/PB12)
- net CAN_TX: now also U109.82 (PD1/CAN1_TX/FSMC_D3/FSMC_DA3); no longer U109.92 (CAN2_TX/DCMI_D5/I2C1_SCL/TIM4_CH1/USART1_TX/PB6)
- net GND: now also R113.2; no longer C112.2
- net at P109.1 (P1), U109.94 (BOOT0): now also R113.1; no longer R113.2
Changed lines of the file:
@@
 Text GLabel 1700 5900 2    60   Input ~ 0
 a7
-Text GLabel 12700 4500 2    60   Input ~ 0
-CAN_TX
-Text GLabel 12700 5100 2    60   Input ~ 0
+Text GLabel 3200 5600 0    60   Input ~ 0
 CAN_RX
 $Comp
@@
 	1250 5800 1450 5800
 Wire Wire Line
-	12450 5100 12700 5100
-Wire Wire Line
-	12700 4500 12450 4500
-Wire Wire Line
 	8250 8700 8400 8700
 Wire Wire Line
@@
 L GND #PWR057
 U 1 1 58942FBF
-P 3050 3400
-F 0 "#PWR057" H 3050 3150 50  0001 C CNN
-F 1 "GND" H 3050 3250 50  0000 C CNN
-F 2 "" H 3050 3400 50  0000 C CNN
-F 3 "" H 3050 3400 50  0000 C CNN
-	1    3050 3400
+P 2500 2850
+F 0 "#PWR057" H 2500 2600 50  0001 C CNN
+F 1 "GND" H 2500 2700 50  0000 C CNN
+F 2 "" H 2500 2850 50  0000 C CNN
+F 3 "" H 2500 2850 50  0000 C CNN
+	1    2500 2850
 	1    0    0    -1
 $EndComp
@@
 Wire Wire Line
 	2700 2300 2700 1750
-Wire Wire Line
-	2500 1750 2800 1750
-Connection ~ 2800 1750
 $Comp
 L CONN_01X06 P110
@@
 L R R113
 U 1 1 588FBA7E
-P 2500 1950
-F 0 "R113" V 2580 1950 50  0000 C CNN
-F 1 "10k" V 2500 1950 50  0000 C CNN
-F 2 "Resistors_SMD:R_0603_HandSoldering" V 2430 1950 50  0001 C CNN
-F 3 "" H 2500 1950 50  0000 C CNN
-	1    2500 1950
-	1    0    0    -1
-$EndComp
-Wire Wire Line
-	2500 2100 2500 2400
-Connection ~ 2500 2400
-Wire Wire Line
-	2500 1800 2500 1750
-Connection ~ 2700 1750
+P 2500 2650
+F 0 "R113" V 2580 2650 50  0000 C CNN
+F 1 "10k" V 2500 2650 50  0000 C CNN
+F 2 "Resistors_SMD:R_0603_HandSoldering" V 2430 2650 50  0001 C CNN
+F 3 "" H 2500 2650 50  0000 C CNN
+	1    2500 2650
+	1    0    0    -1
+$EndComp
 NoConn ~ 15050 5350
 NoConn ~ 12450 3900
@@
 NoConn ~ 3450 4700
 NoConn ~ 3450 4800
-NoConn ~ 3450 5700
 NoConn ~ 3450 5800
 NoConn ~ 3450 5900
@@
 Wire Wire Line
 	12300 8450 12150 8450
-NoConn ~ 3450 5600
 $Comp
 L R R118
@@
 	0    1    1    0
 $EndComp
+Wire Wire Line
+	3450 5600 3200 5600
+Wire Wire Line
+	3200 5700 3450 5700
+Text GLabel 3200 5700 0    60   Input ~ 0
+CAN_TX
+NoConn ~ 12450 4500
+NoConn ~ 12450 5100
+Wire Wire Line
+	2700 1750 2800 1750
+Connection ~ 2800 1750
+Wire Wire Line
+	2500 2850 2500 2800
+Wire Wire Line
+	2500 2500 2500 2400
+Connection ~ 2500 2400
 $EndSCHEMATC

Commit message: erc & drc
Connections:
- net GND: now also C112.2
Changed lines of the file:
@@
 	19300 10050 19300 10650
 Wire Wire Line
-	19400 10550 19950 10550
-Wire Wire Line
-	19500 10450 19950 10450
-Wire Wire Line
-	19950 10250 19550 10250
-Wire Wire Line
 	19550 10250 19550 10300
 Wire Wire Line
@@
 Wire Wire Line
 	18550 9950 19950 9950
-Wire Wire Line
-	19950 10350 19600 10350
 Wire Wire Line
 	19950 9550 18400 9550
@@
 	2500 2500 2500 2400
 Connection ~ 2500 2400
+$Comp
+L GND #PWR072
+U 1 1 58B59181
+P 3050 3400
+F 0 "#PWR072" H 3050 3150 50  0001 C CNN
+F 1 "GND" H 3050 3250 50  0000 C CNN
+F 2 "" H 3050 3400 50  0000 C CNN
+F 3 "" H 3050 3400 50  0000 C CNN
+	1    3050 3400
+	1    0    0    -1
+$EndComp
+Wire Wire Line
+	19400 10550 19950 10550
+Wire Wire Line
+	19500 10450 19950 10450
+Wire Wire Line
+	19600 10350 19950 10350
+Wire Wire Line
+	19950 10250 19550 10250
 $EndSCHEMATC
