File: wr-rusefi.kicad_pcb (KiCad board)
At the start: 2 copper layers, 94 x 94 mm, 1663 parts, among them P101 USB_OTG, P102 CONN_01X08, P103 CONN_01X08, P104 CONN_01X04, P105 CONN_01X08, P106 CONN_01X08, P107 CONN_01X02, P108 USB_OTG, P109 CONN_01X02, P110 CONN_01X06, Q401 IRF540N, Q402 IRF540N, Q403 IRF540N, Q404 IRF540N, Q405 IRF540N, Q406 IRF540N, U101 ISL89410, U102 ISL89410, U103 FT230XS, U104 MAX9924, U105 MCP2562-E/SN, U106 LD1117S33TR, U107 MAX9924, U108 ISL89410, U109 STM32F407VGTx, U110 ISL89410, U201 LM324, U301 LM324, U501 LM7805CT, Y101 Crystal

Commit message: more vias
Parts:
- removed the REF** at (125.7, 116.8)
- removed the REF** at (106.7, 137.2)
- removed the REF** at (120.7, 121.9)
- removed the REF** at (110.5, 139.7)
- removed the REF** at (78.7, 101.6)
- removed the REF** at (77.5, 100.3)
- removed the REF** at (76.2, 106.7)
- removed the REF** at (76.2, 104.1)
- removed the REF** at (83.8, 101.6)
- removed the REF** at (82.5, 101.6)
- removed the REF** at (81.3, 101.6)
- removed the REF** at (80.0, 101.6)
- removed the REF** at (80.0, 100.3)
- removed the REF** at (78.7, 100.3)
- removed the REF** at (105.4, 141.0)
- added REF**: via-stitch, wr-efi:via-stitch, F.Cu at (75.6, 106.7)
- added REF**: via-stitch, wr-efi:via-stitch, F.Cu at (131.4, 127.0)
- added REF**: via-stitch, wr-efi:via-stitch, F.Cu at (131.4, 129.5)
- added REF**: via-stitch, wr-efi:via-stitch, F.Cu at (131.4, 128.3)
- added REF**: via-stitch, wr-efi:via-stitch, F.Cu at (131.4, 130.8)
- added REF**: via-stitch, wr-efi:via-stitch, F.Cu at (131.4, 123.2)
- added REF**: via-stitch, wr-efi:via-stitch, F.Cu at (131.4, 124.5)
- added REF**: via-stitch, wr-efi:via-stitch, F.Cu at (131.4, 120.7)
- added REF**: via-stitch, wr-efi:via-stitch, F.Cu at (131.4, 121.9)
- added REF**: via-stitch, wr-efi:via-stitch, F.Cu at (131.4, 119.4)
- added REF**: via-stitch, wr-efi:via-stitch, F.Cu at (131.4, 118.1)
- added REF**: via-stitch, wr-efi:via-stitch, F.Cu at (75.6, 104.1)
- added REF**: via-stitch, wr-efi:via-stitch, F.Cu at (121.3, 121.3)
- added REF**: via-stitch, wr-efi:via-stitch, F.Cu at (120.0, 121.3)
- added REF**: via-stitch, wr-efi:via-stitch, F.Cu at (120.0, 122.6)
- added REF**: via-stitch, wr-efi:via-stitch, F.Cu at (106.0, 120.0)
- added REF**: via-stitch, wr-efi:via-stitch, F.Cu at (104.8, 122.6)
- added REF**: via-stitch, wr-efi:via-stitch, F.Cu at (109.9, 140.3)
- added REF**: via-stitch, wr-efi:via-stitch, F.Cu at (107.3, 136.5)
- added REF**: via-stitch, wr-efi:via-stitch, F.Cu at (107.3, 135.3)
- added REF**: via-stitch, wr-efi:via-stitch, F.Cu at (107.3, 134.0)
- added REF**: via-stitch, wr-efi:via-stitch, F.Cu at (107.3, 132.7)
- added REF**: via-stitch, wr-efi:via-stitch, F.Cu at (75.6, 101.6)
- added REF**: via-stitch, wr-efi:via-stitch, F.Cu at (107.3, 131.4)
- added REF**: via-stitch, wr-efi:via-stitch, F.Cu at (107.3, 130.2)
- added REF**: via-stitch, wr-efi:via-stitch, F.Cu at (104.8, 130.2)
- added REF**: via-stitch, wr-efi:via-stitch, F.Cu at (97.8, 135.3)
- added REF**: via-stitch, wr-efi:via-stitch, F.Cu at (99.1, 135.3)
- added REF**: via-stitch, wr-efi:via-stitch, F.Cu at (100.3, 135.3)
- added REF**: via-stitch, wr-efi:via-stitch, F.Cu at (100.3, 127.6)
- added REF**: via-stitch, wr-efi:via-stitch, F.Cu at (99.1, 127.6)
- added REF**: via-stitch, wr-efi:via-stitch, F.Cu at (97.8, 127.6)
- added REF**: via-stitch, wr-efi:via-stitch, F.Cu at (90.8, 121.3)
- added REF**: via-stitch, wr-efi:via-stitch, F.Cu at (132.1, 135.9)
- added REF**: via-stitch, wr-efi:via-stitch, F.Cu at (76.8, 100.3)
- added REF**: via-stitch, wr-efi:via-stitch, F.Cu at (78.1, 100.3)
- added REF**: via-stitch, wr-efi:via-stitch, F.Cu at (79.4, 100.3)
- added REF**: via-stitch, wr-efi:via-stitch, F.Cu at (78.1, 101.6)
- added REF**: via-stitch, wr-efi:via-stitch, F.Cu at (79.4, 101.6)
- added REF**: via-stitch, wr-efi:via-stitch, F.Cu at (83.2, 101.0)
- added REF**: via-stitch, wr-efi:via-stitch, F.Cu at (81.9, 101.0)
- added REF**: via-stitch, wr-efi:via-stitch, F.Cu at (80.6, 101.0)
- added REF**: via-stitch, wr-efi:via-stitch, F.Cu at (80.6, 102.2)
- added REF**: via-stitch, wr-efi:via-stitch, F.Cu at (81.9, 102.2)
- added REF**: via-stitch, wr-efi:via-stitch, F.Cu at (131.4, 116.8)
- added REF**: via-stitch, wr-efi:via-stitch, F.Cu at (83.2, 102.2)
- added REF**: via-stitch, wr-efi:via-stitch, F.Cu at (84.5, 102.2)
- added REF**: via-stitch, wr-efi:via-stitch, F.Cu at (85.7, 102.2)
- added REF**: via-stitch, wr-efi:via-stitch, F.Cu at (87.0, 102.2)
- added REF**: via-stitch, wr-efi:via-stitch, F.Cu at (88.3, 102.2)
- added REF**: via-stitch, wr-efi:via-stitch, F.Cu at (89.5, 102.2)
- added REF**: via-stitch, wr-efi:via-stitch, F.Cu at (90.8, 102.2)
- added REF**: via-stitch, wr-efi:via-stitch, F.Cu at (131.4, 125.7)
- added REF**: via-stitch, wr-efi:via-stitch, F.Cu at (131.4, 133.3)
- added REF**: via-stitch, wr-efi:via-stitch, F.Cu at (131.4, 132.1)
- added REF**: via-stitch, wr-efi:via-stitch, F.Cu at (131.4, 134.6)
- moved REF** 2.01 mm to (107.3, 137.8)
- moved REF** 0.90 mm to (106.0, 137.8)
- moved REF** 0.90 mm to (103.5, 137.8)
- moved REF** 0.90 mm to (122.6, 120.0)
- moved REF** 0.90 mm to (125.1, 117.5)
- moved REF** 0.90 mm to (101.0, 121.3)
- moved REF** 0.90 mm to (97.2, 121.3)
- moved REF** 0.90 mm to (95.9, 121.3)
- moved REF** 0.90 mm to (93.3, 121.3)
- moved REF** 0.90 mm to (92.1, 121.3)
- moved REF** 0.90 mm to (92.1, 120.0)
- moved REF** 0.90 mm to (93.3, 120.0)
- moved REF** 0.90 mm to (95.9, 120.0)
- moved REF** 0.90 mm to (97.2, 120.0)
- moved REF** 0.90 mm to (101.0, 120.0)
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Routing:
- net +3V3: track 88.3 -> 88.8 mm
