File: wr-rusefi.kicad_pcb (KiCad board)
At the start: 2 copper layers, 94 x 94 mm, 1704 parts, among them P101 USB_OTG, P102 CONN_01X08, P103 CONN_01X08, P104 CONN_01X04, P105 CONN_01X08, P106 CONN_01X08, P107 CONN_01X02, P108 USB_OTG, P109 CONN_01X02, P110 CONN_01X06, Q401 IRF540N, Q402 IRF540N, Q403 IRF540N, Q404 IRF540N, Q405 IRF540N, Q406 IRF540N, U101 ISL89410, U102 ISL89410, U103 FT230XS, U104 MAX9924, U105 MCP2562-E/SN, U106 LD1117S33TR, U107 MAX9924, U108 ISL89410, U109 STM32F407VGTx, U110 ISL89410, U201 LM324, U301 LM324, U501 LM7805CT, Y101 Crystal

Commit message: erc & drc
Parts:
- removed the REF** at (102.9, 76.2)
- removed the REF** at (99.1, 74.9)
- removed the REF** at (102.9, 74.9)
- removed the REF** at (101.6, 74.9)
- removed the REF** at (100.3, 74.9)
- removed the REF** at (88.9, 81.3)
- removed the REF** at (90.2, 81.3)
- removed the REF** at (91.4, 81.3)
- removed the REF** at (91.4, 82.5)
- removed the REF** at (90.2, 82.5)
- removed the REF** at (88.9, 82.5)
- removed the REF** at (90.2, 83.8)
- removed the REF** at (88.9, 83.8)
- removed the REF** at (91.4, 83.8)
- removed the REF** at (91.4, 86.4)
- removed the REF** at (90.2, 86.4)
- removed the REF** at (88.9, 86.4)
- removed the REF** at (88.9, 85.1)
- removed the REF** at (90.2, 85.1)
- removed the REF** at (91.4, 85.1)
- removed the REF** at (91.4, 87.6)
- removed the REF** at (90.2, 87.6)
- removed the REF** at (88.9, 87.6)
- removed the REF** at (91.4, 88.9)
- removed the REF** at (91.4, 90.2)
- removed the REF** at (90.2, 90.2)
- removed the REF** at (90.2, 88.9)
- removed the REF** at (88.9, 88.9)
- removed the REF** at (88.9, 90.2)
- removed the REF** at (91.4, 91.4)
- removed the REF** at (91.4, 92.7)
- removed the REF** at (90.2, 92.7)
- removed the REF** at (90.2, 91.4)
- removed the REF** at (88.9, 91.4)
- removed the REF** at (88.9, 92.7)
- removed the REF** at (91.4, 94.0)
- removed the REF** at (90.2, 94.0)
- removed the REF** at (88.9, 94.0)
- removed the REF** at (88.9, 95.2)
- removed the REF** at (90.2, 95.2)
- removed the REF** at (91.4, 95.2)
- removed the REF** at (91.4, 96.5)
- removed the REF** at (91.4, 97.8)
- removed the REF** at (90.2, 97.8)
- removed the REF** at (90.2, 96.5)
- removed the REF** at (88.9, 96.5)
- removed the REF** at (88.9, 97.8)
- removed the REF** at (88.9, 114.3)
- removed the REF** at (116.8, 104.1)
- removed the REF** at (101.6, 62.2)
- removed the REF** at (100.3, 67.3)
- added REF**: via-stitch, wr-efi:via-stitch, F.Cu at (102.2, 75.6)
- added REF**: via-stitch, wr-efi:via-stitch, F.Cu at (90.2, 94.6)
- added REF**: via-stitch, wr-efi:via-stitch, F.Cu at (91.4, 94.6)
- added REF**: via-stitch, wr-efi:via-stitch, F.Cu at (90.2, 92.1)
- added REF**: via-stitch, wr-efi:via-stitch, F.Cu at (91.4, 92.1)
- added REF**: via-stitch, wr-efi:via-stitch, F.Cu at (88.9, 84.5)
- added REF**: via-stitch, wr-efi:via-stitch, F.Cu at (88.9, 81.9)
- added REF**: via-stitch, wr-efi:via-stitch, F.Cu at (88.9, 87.0)
- added REF**: via-stitch, wr-efi:via-stitch, F.Cu at (90.2, 84.5)
- added REF**: via-stitch, wr-efi:via-stitch, F.Cu at (90.2, 81.9)
- added REF**: via-stitch, wr-efi:via-stitch, F.Cu at (90.2, 87.0)
- added REF**: via-stitch, wr-efi:via-stitch, F.Cu at (88.9, 97.2)
- added REF**: via-stitch, wr-efi:via-stitch, F.Cu at (91.4, 84.5)
- added REF**: via-stitch, wr-efi:via-stitch, F.Cu at (91.4, 81.9)
- added REF**: via-stitch, wr-efi:via-stitch, F.Cu at (91.4, 87.0)
- added REF**: via-stitch, wr-efi:via-stitch, F.Cu at (114.3, 94.6)
- added REF**: via-stitch, wr-efi:via-stitch, F.Cu at (75.6, 79.4)
- added REF**: via-stitch, wr-efi:via-stitch, F.Cu at (80.0, 79.4)
- added REF**: via-stitch, wr-efi:via-stitch, F.Cu at (78.7, 79.4)
- added REF**: via-stitch, wr-efi:via-stitch, F.Cu at (82.5, 79.4)
- added REF**: via-stitch, wr-efi:via-stitch, F.Cu at (81.3, 79.4)
- added REF**: via-stitch, wr-efi:via-stitch, F.Cu at (85.1, 79.4)
- added REF**: via-stitch, wr-efi:via-stitch, F.Cu at (91.4, 97.2)
- added REF**: via-stitch, wr-efi:via-stitch, F.Cu at (83.8, 79.4)
- added REF**: via-stitch, wr-efi:via-stitch, F.Cu at (87.6, 79.4)
- added REF**: via-stitch, wr-efi:via-stitch, F.Cu at (86.4, 79.4)
- added REF**: via-stitch, wr-efi:via-stitch, F.Cu at (85.7, 96.5)
- added REF**: via-stitch, wr-efi:via-stitch, F.Cu at (85.7, 92.7)
- added REF**: via-stitch, wr-efi:via-stitch, F.Cu at (85.7, 91.4)
- added REF**: via-stitch, wr-efi:via-stitch, F.Cu at (85.7, 87.6)
- added REF**: via-stitch, wr-efi:via-stitch, F.Cu at (85.7, 86.4)
- added REF**: via-stitch, wr-efi:via-stitch, F.Cu at (85.7, 81.3)
- added REF**: via-stitch, wr-efi:via-stitch, F.Cu at (85.7, 82.5)
- added REF**: via-stitch, wr-efi:via-stitch, F.Cu at (90.2, 97.2)
- added REF**: via-stitch, wr-efi:via-stitch, F.Cu at (85.7, 83.8)
- added REF**: via-stitch, wr-efi:via-stitch, F.Cu at (85.7, 85.1)
- added REF**: via-stitch, wr-efi:via-stitch, F.Cu at (85.7, 88.9)
- added REF**: via-stitch, wr-efi:via-stitch, F.Cu at (85.7, 90.2)
- added REF**: via-stitch, wr-efi:via-stitch, F.Cu at (85.7, 94.0)
- added REF**: via-stitch, wr-efi:via-stitch, F.Cu at (85.7, 95.2)
- added REF**: via-stitch, wr-efi:via-stitch, F.Cu at (85.7, 97.8)
- added REF**: via-stitch, wr-efi:via-stitch, F.Cu at (88.9, 89.5)
- added REF**: via-stitch, wr-efi:via-stitch, F.Cu at (91.4, 89.5)
- added REF**: via-stitch, wr-efi:via-stitch, F.Cu at (90.2, 89.5)
- added REF**: via-stitch, wr-efi:via-stitch, F.Cu at (88.9, 92.1)
- added REF**: via-stitch, wr-efi:via-stitch, F.Cu at (88.9, 94.6)
- moved REF** 5.12 mm to (88.9, 79.4)
- moved REF** 5.12 mm to (90.2, 79.4)
- moved REF** 0.90 mm to (99.7, 75.6)
- moved REF** 0.90 mm to (98.4, 75.6)
- moved REF** 0.90 mm to (97.2, 75.6)
- moved REF** 0.90 mm to (94.6, 75.6)
- moved REF** 0.90 mm to (93.3, 75.6)
- moved REF** 0.90 mm to (101.0, 75.6)
- moved REF** 0.90 mm to (95.9, 75.6)
- moved REF** 0.90 mm to (92.1, 75.6)
- moved REF** 0.64 mm to (101.6, 78.1)
- moved REF** 0.64 mm to (100.3, 74.3)
- moved REF** 0.64 mm to (101.6, 74.3)
- moved REF** 0.64 mm to (102.9, 74.3)
- moved REF** 0.64 mm to (92.7, 84.5)
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Connections:
- C112 pad 2: Net-(C112-Pad2) -> GND
Routing:
- net +5V: track 322.4 -> 324.1 mm
- net BATT_ADC: vias 0 -> 2
